Commit message: add lidar stl and fix base_link

File: urdf/mecanum3.xacro (robot description, xacro)
@@ -112,4 +112,26 @@
   </collision>
 </link>
+<link name="LiDAR">
+  <inertial>
+    <origin xyz="0.00023 -0.00145 0.00000" rpy="0 0 90"/>
+    <mass value="0.262"/>
+    <inertia ixx="0.112383" ixy="-0.000264" ixz="-0.00000115"
+             iyy="0.124665" iyz="-0.00000044"
+             izz="0.122901"/>
+  </inertial>
+  <visual>
+    <origin xyz="0 0 0" rpy="0 0 0"/>
+    <geometry>
+      <mesh filename="package://mecanumrover_description/meshes/LiDAR.stl"/>
+    </geometry>
+    <material name="dark_grey"/>
+  </visual>
+  <collision>
+    <origin xyz="0 0 0" rpy="0 0 0"/>
+    <geometry>
+      <mesh filename="package://mecanumrover_description/meshes/LiDAR.stl"/>
+    </geometry>
+  </collision>
+</link>
 <joint name="front_left_joint" type="continuous">
   <origin xyz="-0.0875 0.12 0.076" rpy="0 0 0"/>
@@ -136,3 +158,9 @@
   <axis xyz="-1.0 0.0 0.0"/>
 </joint>
+<joint name="LiDAR_joint" type="fixed">
+  <origin xyz="0.0 0.12 0.160" rpy="0 0 ${radians(-90)}"/>
+  <parent link="base_link"/>
+  <child link="LiDAR"/>
+  <axis xyz="1.0 0.0 0.0"/>
+</joint>
 </robot>

Commit message: add lidar stl and fix base_link

File: urdf/mecanum3.xacro (robot description, xacro)
@@ -10,14 +10,14 @@
   <parent link="base_footprint"/>
   <child link="base_link" />
-  <origin xyz="0 0 0" rpy="0 0 ${radians(-90)}"/>
+  <origin xyz="0 0 0.1" rpy="0 0 ${radians(-90)}"/>
 </joint>
 <link name="base_link">
   <inertial>
-    <origin xyz="8.039076182406018e-05 -0.001484050423595346 0.11040223412633365" rpy="0 0 0"/>
+    <origin xyz="8.039076182406018e-05 -0.001484050423595346 0.01040223412633365" rpy="0 0 0"/>
     <mass value="51.54953324093924"/>
     <inertia ixx="0.451406" iyy="0.211369" izz="0.557559" ixy="0.000784" iyz="0.000199" ixz="-0.000134"/>
   </inertial>
   <visual>
-    <origin xyz="0 0 0" rpy="0 0 0"/>
+    <origin xyz="0 0 -0.1" rpy="0 0 0"/>
     <geometry>
       <mesh filename="package://mecanumrover_description/meshes/base_link.stl" scale="0.001 0.001 0.001"/>
@@ -26,5 +26,5 @@
   </visual>
   <collision>
-    <origin xyz="0 0 0" rpy="0 0 0"/>
+    <origin xyz="0 0 -0.1" rpy="0 0 0"/>
     <geometry>
       <mesh filename="package://mecanumrover_description/meshes/base_link.stl" scale="0.001 0.001 0.001"/>
@@ -135,5 +135,5 @@
 </link>
 <joint name="front_left_joint" type="continuous">
-  <origin xyz="-0.0875 0.12 0.076" rpy="0 0 0"/>
+  <origin xyz="-0.0875 0.12 -0.024" rpy="0 0 0"/>
   <parent link="base_link"/>
   <child link="front_left_wheel_1"/>
@@ -141,5 +141,5 @@
 </joint>
 <joint name="front_right_joint" type="continuous">
-  <origin xyz="0.0875 0.12 0.076" rpy="0 0 0"/>
+  <origin xyz="0.0875 0.12 -0.024" rpy="0 0 0"/>
   <parent link="base_link"/>
   <child link="front_right_wheel_1"/>
@@ -147,5 +147,5 @@
 </joint>
 <joint name="back_right_joint" type="continuous">
-  <origin xyz="0.0875 -0.12 0.076" rpy="0 0 0"/>
+  <origin xyz="0.0875 -0.12 -0.024" rpy="0 0 0"/>
   <parent link="base_link"/>
   <child link="back_right_wheel_1"/>
@@ -153,5 +153,5 @@
 </joint>
 <joint name="back_left_joint" type="continuous">
-  <origin xyz="-0.0875 -0.12 0.076" rpy="0 0 0"/>
+  <origin xyz="-0.0875 -0.12 -0.024" rpy="0 0 0"/>
   <parent link="base_link"/>
   <child link="back_left_wheel_1"/>
@@ -159,5 +159,5 @@
 </joint>
 <joint name="LiDAR_joint" type="fixed">
-  <origin xyz="0.0 0.12 0.160" rpy="0 0 ${radians(-90)}"/>
+  <origin xyz="0.0 0.12 0.060" rpy="0 0 ${radians(-90)}"/>
   <parent link="base_link"/>
   <child link="LiDAR"/>

Commit message: fix scale and origin

File: urdf/mecanum3.xacro (robot description, xacro)
@@ -114,5 +114,5 @@
 <link name="LiDAR">
   <inertial>
-    <origin xyz="0.00023 -0.00145 0.00000" rpy="0 0 90"/>
+    <origin xyz="0.00023 -0.00145 0.00000" rpy="0 0 0"/>
     <mass value="0.262"/>
     <inertia ixx="0.112383" ixy="-0.000264" ixz="-0.00000115"
@@ -123,5 +123,5 @@
     <origin xyz="0 0 0" rpy="0 0 0"/>
     <geometry>
-      <mesh filename="package://mecanumrover_description/meshes/LiDAR.stl"/>
+      <mesh filename="package://mecanumrover_description/meshes/mid-360-asm.STL"  scale="0.001 0.001 0.001"/>
     </geometry>
     <material name="dark_grey"/>
@@ -130,5 +130,5 @@
     <origin xyz="0 0 0" rpy="0 0 0"/>
     <geometry>
-      <mesh filename="package://mecanumrover_description/meshes/LiDAR.stl"/>
+      <mesh filename="package://mecanumrover_description/meshes/mid-360-asm.STL"  scale="0.001 0.001 0.001"/>
     </geometry>
   </collision>
@@ -159,5 +159,5 @@
 </joint>
 <joint name="LiDAR_joint" type="fixed">
-  <origin xyz="0.0 0.12 0.060" rpy="0 0 ${radians(-90)}"/>
+  <origin xyz="0.04 0.15 0.060" rpy="${radians(90)} 0 ${radians(-90)}"/>
   <parent link="base_link"/>
   <child link="LiDAR"/>

Commit message: rviz supporting pallet by three ground robot

File: urdf/mecanum3.xacro (robot description, xacro)
@@ -134,4 +134,26 @@
   </collision>
 </link>
+<link name="pillar_and_pc">
+  <inertial>
+    <origin xyz="0.01 0.00 -0.03" rpy="0 0 0"/>
+    <mass value="0.42811"/>
+    <inertia ixx="1.73" ixy="0.09" ixz="-0.13"
+             iyy="2.93" iyz="0.07"
+             izz="3.31"/>
+  </inertial>
+  <visual>
+    <origin xyz="0 0 0" rpy="0 0 0"/>
+    <geometry>
+      <mesh filename="package://mecanumrover_description/meshes/pillar_and_pc.STL"/>
+    </geometry>
+    <material name="dark_grey"/>
+  </visual>
+  <collision>
+    <origin xyz="0 0 0" rpy="0 0 0"/>
+    <geometry>
+      <mesh filename="package://mecanumrover_description/meshes/pillar_and_pc.STL"/>
+    </geometry>
+  </collision>
+</link>
 <joint name="front_left_joint" type="continuous">
   <origin xyz="-0.0875 0.12 -0.024" rpy="0 0 0"/>
@@ -164,3 +186,9 @@
   <axis xyz="1.0 0.0 0.0"/>
 </joint>
+<joint name="pillar_and_pc_joint" type="fixed">
+  <origin xyz="0.0 -0.03 0.1100" rpy="0 0 ${radians(90)}"/>
+  <parent link="base_link"/>
+  <child link="pillar_and_pc"/>
+  <axis xyz="1.0 0.0 0.0"/>
+</joint>
 </robot>
